Commit message: Works now

File: urdf/conveyor.urdf.xacro (robot description, xacro)
@@ -12,5 +12,5 @@
   <xacro:arg name="load_rollers" default="false"/>
   <xacro:arg name="load_motors" default="false"/>
-  <xacro:arg name="load_railings" default="true"/>
+  <xacro:arg name="load_railings" default="false"/>
   <material name="white">
     <color rgba="1 1 1 1"/>
@@ -41,5 +41,5 @@
     <link name="frame" type="fixed" >
        <visual>
-	<origin rpy="0 0 0" xyz="0.75 -0.75 0" />
+	<origin rpy="0 0 0" xyz="0.5 -0.75 0" />
   	  <geometry>
 		<mesh filename="package://ur3e_irl_project/meshes/frame.stl"/>
@@ -47,5 +47,5 @@
        </visual>
 	<collision>
-          <origin rpy="0 0 0" xyz="0.75 -0.75 0" />
+          <origin rpy="0 0 0" xyz="0.5 -0.75 0" />
   	  <geometry>
 		<mesh filename="package://ur3e_irl_project/meshes/conveyor_box.stl"/>
@@ -59,5 +59,5 @@
     </link>
   <joint name="frame_to_belt" type="fixed">
-    <origin rpy="0 0 0" xyz="0.75 0 0.73" />
+    <origin rpy="0 0 0" xyz="0.5 0 0.73" />
     <parent link="frame"/>
     <child link="belt"/>

File: urdf/conveyor_g_path.urdf.xacro (robot description, xacro)
@@ -182,5 +182,5 @@
       </collision>
     </link>
-<!--    <link name="world">
+   <link name="world">
       <inertial>
         <origin xyz="0 0 0" rpy="0 0 0"/>
@@ -193,5 +193,5 @@
     <parent link="world"/>
     <child link="conveyor_base"/>
-  </joint>-->
+  </joint>
     <link name="conveyor_base">
       <inertial>

Commit message: Conveyor corrected

File: urdf/conveyor.urdf.xacro (robot description, xacro)
@@ -43,5 +43,5 @@
 	<origin rpy="0 0 0" xyz="0.75 -0.75 0" />
   	  <geometry>
-		<mesh filename="package://ur3e_irl_project/meshes/frame.stl"/>
+		<mesh filename="package://ur3e_irl_project/meshes/lab_conveyor/frame.stl"/>
 	  </geometry>
        </visual>
@@ -49,5 +49,5 @@
           <origin rpy="0 0 0" xyz="0.75 -0.75 0" />
   	  <geometry>
-		<mesh filename="package://ur3e_irl_project/meshes/conveyor_box.stl"/>
+		<mesh filename="package://ur3e_irl_project/meshes/lab_conveyor/conveyor_box.stl"/>
 	  </geometry>
 	</collision>
@@ -70,5 +70,5 @@
 	<origin rpy="0 0 0" xyz="0 0 0" />
   	  <geometry>
-		<mesh filename="package://ur3e_irl_project/meshes/belt.stl"/>
+		<mesh filename="package://ur3e_irl_project/meshes/lab_conveyor/belt.stl"/>
 	  </geometry>
        </visual>
@@ -76,5 +76,5 @@
           <origin rpy="0 0 0" xyz="0 0 0" />
   	  <geometry>
-		<mesh filename="package://ur3e_irl_project/meshes/belt.stl"/>
+		<mesh filename="package://ur3e_irl_project/meshes/lab_conveyor/belt.stl"/>
 	  </geometry>
 	</collision>
@@ -166,5 +166,5 @@
 	<origin rpy="0 0 0" xyz="0 0 0" />
   	  <geometry>
-		<mesh filename="package://ur3e_irl_project/meshes/roller.stl"/>
+		<mesh filename="package://ur3e_irl_project/meshes/lab_conveyor/roller.stl"/>
 	  </geometry>
        </visual>
@@ -195,5 +195,5 @@
 	<origin rpy="0 0 0" xyz="0 0 0" />
   	  <geometry>
-		<mesh filename="package://ur3e_irl_project/meshes/roller.stl"/>
+		<mesh filename="package://ur3e_irl_project/meshes/lab_conveyor/roller.stl"/>
 	  </geometry>
        </visual>
@@ -224,5 +224,5 @@
 	<origin rpy="0 0 0" xyz="0 0 0" />
   	  <geometry>
-		<mesh filename="package://ur3e_irl_project/meshes/roller.stl"/>
+		<mesh filename="package://ur3e_irl_project/meshes/lab_conveyor/roller.stl"/>
 	  </geometry>
        </visual>
@@ -253,5 +253,5 @@
 	    <origin rpy="0 0 0" xyz="0 0 0" />
   	  <geometry>
-		  <mesh filename="package://ur3e_irl_project/meshes/roller.stl"/>
+		  <mesh filename="package://ur3e_irl_project/meshes/lab_conveyor/roller.stl"/>
 	    </geometry>
       </visual>
@@ -282,5 +282,5 @@
 	<origin rpy="0 0 0" xyz="0 0 0" />
   	  <geometry>
-		<mesh filename="package://ur3e_irl_project/meshes/roller.stl"/>
+		<mesh filename="package://ur3e_irl_project/meshes/lab_conveyor/roller.stl"/>
 	  </geometry>
        </visual>
@@ -311,5 +311,5 @@
 	<origin rpy="0 0 0" xyz="0 0 0" />
   	  <geometry>
-		<mesh filename="package://ur3e_irl_project/meshes/roller.stl"/>
+		<mesh filename="package://ur3e_irl_project/meshes/lab_conveyor/roller.stl"/>
 	  </geometry>
        </visual>
@@ -340,5 +340,5 @@
 	<origin rpy="0 0 0" xyz="0 0 0" />
   	  <geometry>
-		<mesh filename="package://ur3e_irl_project/meshes/roller.stl"/>
+		<mesh filename="package://ur3e_irl_project/meshes/lab_conveyor/roller.stl"/>
 	  </geometry>
        </visual>
@@ -369,5 +369,5 @@
 	<origin rpy="0 0 0" xyz="0 0 0" />
   	  <geometry>
-		<mesh filename="package://ur3e_irl_project/meshes/roller.stl"/>
+		<mesh filename="package://ur3e_irl_project/meshes/lab_conveyor/roller.stl"/>
 	  </geometry>
        </visual>
@@ -398,5 +398,5 @@
 	<origin rpy="0 0 0" xyz="0 0 0" />
   	  <geometry>
-		<mesh filename="package://ur3e_irl_project/meshes/roller.stl"/>
+		<mesh filename="package://ur3e_irl_project/meshes/lab_conveyor/roller.stl"/>
 	  </geometry>
        </visual>
@@ -427,5 +427,5 @@
 	<origin rpy="0 0 0" xyz="0 0 0" />
   	  <geometry>
-		<mesh filename="package://ur3e_irl_project/meshes/roller.stl"/>
+		<mesh filename="package://ur3e_irl_project/meshes/lab_conveyor/roller.stl"/>
 	  </geometry>
        </visual>
@@ -456,5 +456,5 @@
 	<origin rpy="0 0 0" xyz="0 0 0" />
   	  <geometry>
-		<mesh filename="package://ur3e_irl_project/meshes/roller.stl"/>
+		<mesh filename="package://ur3e_irl_project/meshes/lab_conveyor/roller.stl"/>
 	  </geometry>
        </visual>
@@ -485,5 +485,5 @@
 	<origin rpy="0 0 0" xyz="0 0 0" />
   	  <geometry>
-		<mesh filename="package://ur3e_irl_project/meshes/roller.stl"/>
+		<mesh filename="package://ur3e_irl_project/meshes/lab_conveyor/roller.stl"/>
 	  </geometry>
        </visual>
@@ -514,5 +514,5 @@
 	<origin rpy="0 0 0" xyz="0 0 0" />
   	  <geometry>
-		<mesh filename="package://ur3e_irl_project/meshes/roller.stl"/>
+		<mesh filename="package://ur3e_irl_project/meshes/lab_conveyor/roller.stl"/>
 	  </geometry>
        </visual>
@@ -543,5 +543,5 @@
 	<origin rpy="0 0 0" xyz="0 0 0" />
   	  <geometry>
-		<mesh filename="package://ur3e_irl_project/meshes/roller.stl"/>
+		<mesh filename="package://ur3e_irl_project/meshes/lab_conveyor/roller.stl"/>
 	  </geometry>
        </visual>
@@ -572,5 +572,5 @@
 	<origin rpy="0 0 0" xyz="0 0 0" />
   	  <geometry>
-		<mesh filename="package://ur3e_irl_project/meshes/roller.stl"/>
+		<mesh filename="package://ur3e_irl_project/meshes/lab_conveyor/roller.stl"/>
 	  </geometry>
        </visual>
@@ -601,5 +601,5 @@
 	<origin rpy="0 0 0" xyz="0 0 0" />
   	  <geometry>
-		<mesh filename="package://ur3e_irl_project/meshes/roller.stl"/>
+		<mesh filename="package://ur3e_irl_project/meshes/lab_conveyor/roller.stl"/>
 	  </geometry>
        </visual>

File: urdf/conveyor_g_path.urdf.xacro (robot description, xacro)
@@ -1,23 +1,24 @@
 <?xml version="1.0"?>
 <!-- created with Phobos 1.0.1 "Capricious Choutengan" -->
-  <robot name="conveyor_g">
+  <robot name="conveyor_g" xmlns:xacro="http://www.ros.org/wiki/xacro">
     <link name="link_belt">
       <inertial>
         <origin xyz="0 0 0" rpy="0 0 0"/>
-        <mass value="10.0"/>
-        <inertia ixx="0.38299" ixy="0" ixz="0" iyy="31.09613" iyz="0" izz="31.47895"/>
+        <mass value="0.001"/>
+        <inertia ixx="0.001" ixy="0" ixz="0" iyy="0.001" iyz="0" izz="0.001"/>
       </inertial>
       <visual name="visual_belt">
         <origin xyz="0 0 0" rpy="0 0 0"/>
         <geometry>
-          <mesh filename="package://ur3e_irl_project/meshes/belt.dae" scale="1.0 1.0 1.0"/>
+          <mesh filename="package://ur3e_irl_project/meshes/vovrc_conveyor/belt.dae" scale="0.001 0.001 0.001"/>
         </geometry>
-        <material name="5,5,5"/>
+        <material name="191,191,191"/>
       </visual>
-      <collision name="collision_belt">
+      <collision name="visual_belt">
         <origin xyz="0 0 0" rpy="0 0 0"/>
         <geometry>
-          <box size="6.10862 0.67785 0.01"/>
+          <mesh filename="package://ur3e_irl_project/meshes/vovrc_conveyor/belt.dae" scale="0.001 0.001 0.001"/>
         </geometry>
+        <material name="191,191,191"/>
       </collision>
     </link>
@@ -25,162 +26,16 @@
       <inertial>
         <origin xyz="0 0 0" rpy="0 0 0"/>
-        <mass value="10.0"/>
-        <inertia ixx="0.49874" ixy="0" ixz="0" iyy="0.01319" iyz="0" izz="0.48632"/>
+        <mass value="0.001"/>
+        <inertia ixx="0.001" ixy="0" ixz="0" iyy="0.001" iyz="0" izz="0.001"/>
       </inertial>
       <visual name="visual_bridge_left">
         <origin xyz="0 0 0" rpy="0 0 0"/>
         <geometry>
-          <mesh filename="package://ur3e_irl_project/meshes/bridge_left.dae" scale="1.0 1.0 1.0"/>
+          <mesh filename="package://ur3e_irl_project/meshes/vovrc_conveyor/bridge_left.dae" scale="0.001 0.001 0.001"/>
         </geometry>
         <material name="191,191,191"/>
       </visual>
-      <collision name="collision_bridge_left">
-        <origin xyz="0 0 0.00635" rpy="0 0 0"/>
-        <geometry>
-          <box size="0.0254 0.67785 0.127"/>
-        </geometry>
-      </collision>
     </link>
     <link name="link_bridge_right">
-      <inertial>
-        <origin xyz="0 0 0" rpy="0 0 0"/>
-        <mass value="10.0"/>
-        <inertia ixx="0.49874" ixy="0" ixz="0" iyy="0.01319" iyz="0" izz="0.48632"/>
-      </inertial>
-      <visual name="visual_bridge_right">
-        <origin xyz="0 0 0" rpy="0 0 0"/>
-        <geometry>
-          <mesh filename="package://ur3e_irl_project/meshes/brigde_right.dae" scale="1.0 1.0 1.0"/>
-        </geometry>
-        <material name="191,191,191"/>
-      </visual>
-      <collision name="collision_bridge_right">
-        <origin xyz="0 0 0.00635" rpy="0 0 0"/>
-        <geometry>
-          <box size="0.0254 0.67785 0.127"/>
-        </geometry>
-      </collision>
-    </link>
-    <link name="link_flap_back">
-      <inertial>
-        <origin xyz="0 0 0" rpy="0 0 0"/>
-        <mass value="10.0"/>
-        <inertia ixx="0.00593" ixy="0" ixz="0" iyy="31.1013" iyz="0" izz="31.09673"/>
-      </inertial>
-      <visual name="visual_flap_back">
-        <origin xyz="0 0 0" rpy="0 0 0"/>
-        <geometry>
-          <mesh filename="package://ur3e_irl_project/meshes/flap_back.dae" scale="1.0 1.0 1.0"/>
-        </geometry>
-        <material name="191,191,191"/>
-      </visual>
-      <collision name="collision_flap_back">
-        <origin xyz="0 0 0" rpy="0 0 0"/>
-        <geometry>
-          <box size="6.10862 0.02857 0.07937"/>
-        </geometry>
-      </collision>
-    </link>
-    <link name="link_flap_front">
-      <inertial>
-        <origin xyz="0 0 0" rpy="0 0 0"/>
-        <mass value="10.0"/>
-        <inertia ixx="0.00593" ixy="0" ixz="0" iyy="31.1013" iyz="0" izz="31.09673"/>
-      </inertial>
-      <visual name="visual_flap_front">
-        <origin xyz="0 0 0" rpy="0 0 0"/>
-        <geometry>
-          <mesh filename="package://ur3e_irl_project/meshes/flap_front.dae" scale="1.0 1.0 1.0"/>
-        </geometry>
-        <material name="191,191,191"/>
-      </visual>
-      <collision name="collision_flap_front">
-        <origin xyz="0 0 0" rpy="0 0 0"/>
-        <geometry>
-          <box size="6.10862 0.02857 0.07937"/>
-        </geometry>
-      </collision>
-    </link>
-    <link name="link_leg_back_left">
-      <inertial>
-        <origin xyz="0 0 0" rpy="0 0 0"/>
-        <mass value="10.0"/>
-        <inertia ixx="1.29297" ixy="0" ixz="0" iyy="1.29297" iyz="0" izz="0.0043"/>
-      </inertial>
-      <visual name="visual_leg_back_left">
-        <origin xyz="0 0 0" rpy="0 0 0"/>
-        <geometry>
-          <mesh filename="package://ur3e_irl_project/meshes/leg_back_left.dae" scale="1.0 1.0 1.0"/>
-        </geometry>
-        <material name="191,191,191"/>
-      </visual>
-      <collision name="collision_leg_back_left">
-        <origin xyz="0 0 0" rpy="0 0 0"/>
-        <geometry>
-          <box size="0.0508 0.0508 1.24458"/>
-        </geometry>
-      </collision>
-    </link>
-    <link name="link_leg_back_right">
-      <inertial>
-        <origin xyz="0 0 0" rpy="0 0 0"/>
-        <mass value="10.0"/>
-        <inertia ixx="1.29297" ixy="0" ixz="0" iyy="1.29297" iyz="0" izz="0.0043"/>
-      </inertial>
-      <visual name="visual_leg_back_right">
-        <origin xyz="0 0 0" rpy="0 0 0"/>
-        <geometry>
-          <mesh filename="package://ur3e_irl_project/meshes/leg_back_right.dae" scale="1.0 1.0 1.0"/>
-        </geometry>
-        <material name="191,191,191"/>
-      </visual>
-      <collision name="collision_leg_back_right">
-        <origin xyz="0 0 0" rpy="0 0 0"/>
-        <geometry>
-          <box size="0.0508 0.0508 1.24458"/>
-        </geometry>
-      </collision>
-    </link>
-    <link name="link_leg_front_left">
-      <inertial>
-        <origin xyz="0 0 0" rpy="0 0 0"/>
-        <mass value="10.0"/>
-        <inertia ixx="1.29297" ixy="0" ixz="0" iyy="1.29297" iyz="0" izz="0.0043"/>
-      </inertial>
-      <visual name="visual_leg_front_left">
-        <origin xyz="0 0 0" rpy="0 0 0"/>
-        <geometry>
-          <mesh filename="package://ur3e_irl_project/meshes/leg_front_left.dae" scale="1.0 1.0 1.0"/>
-        </geometry>
-        <material name="191,191,191"/>
-      </visual>
-      <collision name="collision_leg_front_left">
-        <origin xyz="0 0 0" rpy="0 0 0"/>
-        <geometry>
-          <box size="0.0508 0.0508 1.24458"/>
-        </geometry>
-      </collision>
-    </link>
-    <link name="link_leg_front_right">
-      <inertial>
-        <origin xyz="0 0 0" rpy="0 0 0"/>
-        <mass value="10.0"/>
-        <inertia ixx="1.29297" ixy="0" ixz="0" iyy="1.29297" iyz="0" izz="0.0043"/>
-      </inertial>
-      <visual name="visual_leg_front_right">
-        <origin xyz="0 0 0" rpy="0 0 0"/>
-        <geometry>
-          <mesh filename="package://ur3e_irl_project/meshes/leg_front_right.dae" scale="1.0 1.0 1.0"/>
-        </geometry>
-        <material name="191,191,191"/>
-      </visual>
-      <collision name="collision_leg_front_right">
-        <origin xyz="0 0 0" rpy="0 0 0"/>
-        <geometry>
-          <box size="0.0508 0.0508 1.24458"/>
-        </geometry>
-      </collision>
-    </link>
-<!--    <link name="world">
       <inertial>
         <origin xyz="0 0 0" rpy="0 0 0"/>
@@ -188,11 +43,97 @@
         <inertia ixx="0.001" ixy="0" ixz="0" iyy="0.001" iyz="0" izz="0.001"/>
       </inertial>
+      <visual name="visual_bridge_right">
+        <origin xyz="0 0 0" rpy="0 0 0"/>
+        <geometry>
+          <mesh filename="package://ur3e_irl_project/meshes/vovrc_conveyor/bridge_right.dae" scale="0.001 0.001 0.001"/>
+        </geometry>
+        <material name="191,191,191"/>
+      </visual>
     </link>
-  <joint name="world_to_conveyor_base" type="fixed">
-    <origin xyz="0 0 0" rpy="0 0 0"/>
-    <parent link="world"/>
-    <child link="conveyor_base"/>
-  </joint>-->
-    <link name="conveyor_base">
+    <link name="link_flap_back">
+      <inertial>
+        <origin xyz="0 0 0" rpy="0 0 0"/>
+        <mass value="0.001"/>
+        <inertia ixx="0.001" ixy="0" ixz="0" iyy="0.001" iyz="0" izz="0.001"/>
+      </inertial>
+      <visual name="visual_back_flap">
+        <origin xyz="0 0 0" rpy="0 0 0"/>
+        <geometry>
+          <mesh filename="package://ur3e_irl_project/meshes/vovrc_conveyor/flap_back.dae" scale="0.001 0.001 0.001"/>
+        </geometry>
+        <material name="191,191,191"/>
+      </visual>
+    </link>
+    <link name="link_flap_front">
+      <inertial>
+        <origin xyz="0 0 0" rpy="0 0 0"/>
+        <mass value="0.001"/>
+        <inertia ixx="0.001" ixy="0" ixz="0" iyy="0.001" iyz="0" izz="0.001"/>
+      </inertial>
+      <visual name="visual_flap_front">
+        <origin xyz="0 0 0" rpy="0 0 0"/>
+        <geometry>
+          <mesh filename="package://ur3e_irl_project/meshes/vovrc_conveyor/flap_front.dae" scale="0.001 0.001 0.001"/>
+        </geometry>
+        <material name="191,191,191"/>
+      </visual>
+    </link>
+    <link name="link_leg_back_left">
+      <inertial>
+        <origin xyz="0 0 0" rpy="0 0 0"/>
+        <mass value="0.001"/>
+        <inertia ixx="0.001" ixy="0" ixz="0" iyy="0.001" iyz="0" izz="0.001"/>
+      </inertial>
+      <visual name="visual_leg_back_left">
+        <origin xyz="0 0 0" rpy="0 0 0"/>
+        <geometry>
+          <mesh filename="package://ur3e_irl_project/meshes/vovrc_conveyor/leg_back_left.dae" scale="0.001 0.001 0.001"/>
+        </geometry>
+        <material name="191,191,191"/>
+      </visual>
+    </link>
+    <link name="link_leg_back_right">
+      <inertial>
+        <origin xyz="0 0 0" rpy="0 0 0"/>
+        <mass value="0.001"/>
+        <inertia ixx="0.001" ixy="0" ixz="0" iyy="0.001" iyz="0" izz="0.001"/>
+      </inertial>
+      <visual name="visual_leg_back_right">
+        <origin xyz="0 0 0" rpy="0 0 0"/>
+        <geometry>
+          <mesh filename="package://ur3e_irl_project/meshes/vovrc_conveyor/leg_back_right.dae" scale="0.001 0.001 0.001"/>
+        </geometry>
+        <material name="191,191,191"/>
+      </visual>
+    </link>
+    <link name="link_leg_front_left">
+      <inertial>
+        <origin xyz="0 0 0" rpy="0 0 0"/>
+        <mass value="0.001"/>
+        <inertia ixx="0.001" ixy="0" ixz="0" iyy="0.001" iyz="0" izz="0.001"/>
+      </inertial>
+      <visual name="visual_leg_front_left">
+        <origin xyz="0 0 0" rpy="0 0 0"/>
+        <geometry>
+          <mesh filename="package://ur3e_irl_project/meshes/vovrc_conveyor/leg_front_left.dae" scale="0.001 0.001 0.001"/>
+        </geometry>
+        <material name="191,191,191"/>
+      </visual>
+    </link>
+    <link name="link_leg_front_right">
+      <inertial>
+        <origin xyz="0 0 0" rpy="0 0 0"/>
+        <mass value="0.001"/>
+        <inertia ixx="0.001" ixy="0" ixz="0" iyy="0.001" iyz="0" izz="0.001"/>
+      </inertial>
+      <visual name="visual_leg_front_right">
+        <origin xyz="0 0 0" rpy="0 0 0"/>
+        <geometry>
+          <mesh filename="package://ur3e_irl_project/meshes/vovrc_conveyor/leg_front_right.dae" scale="0.001 0.001 0.001"/>
+        </geometry>
+        <material name="191,191,191"/>
+      </visual>
+    </link>
+    <link name="world">
       <inertial>
         <origin xyz="0 0 0" rpy="0 0 0"/>
@@ -202,46 +143,46 @@
     </link>
     <joint name="joint_belt" type="fixed">
-      <origin xyz="0 0.33893 -0.08438" rpy="0 0 0"/>
-      <parent link="conveyor_base"/>
+      <origin xyz="0 0.3048 1.07" rpy="0 0 0"/>
+      <parent link="world"/>
       <child link="link_belt"/>
     </joint>
     <joint name="joint_bridge_left" type="fixed">
-      <origin xyz="0.62864 0.33893 0.05714" rpy="0 0 0"/>
-      <parent link="conveyor_base"/>
+      <origin xyz="0.59689 0.3048 1.17414" rpy="0 0 0"/>
+      <parent link="world"/>
       <child link="link_bridge_left"/>
     </joint>
     <joint name="joint_bridge_right" type="fixed">
-      <origin xyz="-1.79703 0.33893 0.05714" rpy="0 0 0"/>
-      <parent link="conveyor_base"/>
+      <origin xyz="-0.85089 0.3048 1.17414" rpy="0 0 0"/>
+      <parent link="world"/>
       <child link="link_bridge_right"/>
     </joint>
     <joint name="joint_flap_back" type="fixed">
-      <origin xyz="0 0.01429 -0.03969" rpy="0 0 0"/>
-      <parent link="conveyor_base"/>
+      <origin xyz="0 0.0127 1.096" rpy="0 0 0"/>
+      <parent link="world"/>
       <child link="link_flap_back"/>
     </joint>
     <joint name="joint_flap_front" type="fixed">
-      <origin xyz="0 0.66357 -0.03969" rpy="0 0 0"/>
-      <parent link="conveyor_base"/>
+      <origin xyz="0 0.59689 1.096" rpy="0 0 0"/>
+      <parent link="world"/>
       <child link="link_flap_front"/>
     </joint>
     <joint name="joint_leg_back_left" type="fixed">
-      <origin xyz="1.68273 -0.0254 -0.6223" rpy="0 0 0"/>
-      <parent link="conveyor_base"/>
+      <origin xyz="0.68579 -0.0254 0.57" rpy="0 0 0"/>
+      <parent link="world"/>
       <child link="link_leg_back_left"/>
     </joint>
     <joint name="joint_leg_back_right" type="fixed">
-      <origin xyz="-1.68273 -0.0254 -0.6223" rpy="0 0 0"/>
-      <parent link="conveyor_base"/>
+      <origin xyz="-0.68579 -0.0254 0.57" rpy="0 0 0"/>
+      <parent link="world"/>
       <child link="link_leg_back_right"/>
     </joint>
     <joint name="joint_leg_front_left" type="fixed">
-      <origin xyz="1.68273 0.70325 -0.6223" rpy="0 0 0"/>
-      <parent link="conveyor_base"/>
+      <origin xyz="0.68579 0.63499 0.57" rpy="0 0 0"/>
+      <parent link="world"/>
       <child link="link_leg_front_left"/>
     </joint>
     <joint name="joint_leg_front_right" type="fixed">
-      <origin xyz="-1.68273 0.70325 -0.6223" rpy="0 0 0"/>
-      <parent link="conveyor_base"/>
+      <origin xyz="-0.68579 0.63499 0.57" rpy="0 0 0"/>
+      <parent link="world"/>
       <child link="link_leg_front_right"/>
     </joint>
@@ -249,6 +190,3 @@
       <color rgba="0.74902 0.74902 0.74902 1.0"/>
     </material>
-    <material name="5,5,5">
-      <color rgba="0.01961 0.01961 0.01961 1.0"/>
-    </material>
   </robot>

File: urdf/ur3e_combined.urdf.xacro (robot description, xacro)
@@ -4,5 +4,5 @@
 <robot name="ur3e" xmlns:xacro="http://www.ros.org/wiki/xacro">
   <xacro:include filename="$(find ur_description)/urdf/ur3e.xacro"/>
-  <xacro:include filename="$(find ur3e_irl_project)/urdf/conveyor_g_path.urdf.xacro"/>
+  <!--xacro:include filename="$(find ur3e_irl_project)/urdf/conveyor_g_path.urdf.xacro"/-->
   <xacro:include filename="$(find ur3e_irl_project)/onrobot_sg/models/onrobot_sg_b/sg_b.urdf"/>
   <link name="world" />
@@ -43,10 +43,10 @@
     <child link="quick_change_robot_side"/>
   </joint>
-  <!-- fix the conveyor belt in place -->
+  <!-- fix the conveyor belt in place >
   <joint name="world_to_conveyor_base" type="fixed">
     <origin xyz="0 0.065 1.26458" rpy="0 0 0"/>
     <parent link="world"/>
     <child link="conveyor_base"/>
-  </joint>
+  </joint-->
   <joint name="fixed" type="fixed">
       <parent link="world"/>
