Commit message: In test

File: urdf/ur3e_combined_gazebo.urdf.xacro (robot description, xacro)
@@ -16,5 +16,5 @@
         <origin xyz="0 0 0" rpy="0 0 0"/>
         <geometry>
-          <box size="0.15 0.15 0.8"/>
+          <box size="0.15 0.15 1.2"/>
         </geometry>
         <material name="4,4,4"/>
@@ -23,5 +23,5 @@
         <origin xyz="0 0 0" rpy="0 0 0"/>
         <geometry>
-          <box size="0.15 0.15 0.8"/>
+          <box size="0.15 0.15 1.2"/>
         </geometry>
       </collision>
@@ -69,5 +69,5 @@
   <!-- fix the ur robot in place -->
   <joint name="world_to_pillar" type="fixed">
-    <origin xyz="0 0 0.4" rpy="0 0 0"/>
+    <origin xyz="0 0 0.6" rpy="0 0 0"/>
     <parent link="world"/>
     <child link="support_pillar"/>
@@ -79,5 +79,5 @@
   </joint-->
   <joint name="pillar_to_base" type="fixed">
-    <origin xyz="0 0 0.4" rpy="0 0 0"/>
+    <origin xyz="0 0 0.6" rpy="0 0 0"/>
     <parent link="support_pillar"/>
     <child link="base_link"/>

Commit message: Fixed gazebo sim

File: urdf/ur3e_combined_gazebo.urdf.xacro (robot description, xacro)
@@ -27,5 +27,5 @@
       </collision>
   </link>
-  <!--link name="rear_pillars">
+  <link name="rear_pillars">
       <inertial>
         <origin xyz="0 0 0" rpy="0 0 0"/>
@@ -46,6 +46,6 @@
         </geometry>
       </collision>
-  </link-->
-  <!-- <link name="vention_assembly">
+  </link>
+   <!-- <link name="vention_assembly">
       <inertial>
         <origin xyz="-1.25 -0.8 0" rpy="1.6 0 0"/>
@@ -73,24 +73,24 @@
     <child link="support_pillar"/>
   </joint>
-  <!--joint name="world_to_assembly" type="fixed">
+  <joint name="pillar_to_base" type="fixed">
+  <origin xyz="0 0 0.6" rpy="0 0 0"/>
+  <parent link="support_pillar"/>
+  <child link="base_link"/>
+  </joint>
+  <joint name="pillar_to_rear_pillars" type="fixed">
+  <origin xyz="0 -0.37 0.8" rpy="0 0 0"/>
+  <parent link="support_pillar"/>
+  <child link="rear_pillars"/>
+</joint>
+  <!-- <joint name="world_to_assembly" type="fixed">
     <origin xyz="0 0 0.0" rpy="0 0 0"/>
     <parent link="world"/>
     <child link="vention_assembly"/>
-  </joint-->
-  <joint name="pillar_to_base" type="fixed">
-    <origin xyz="0 0 0.6" rpy="0 0 0"/>
-    <parent link="support_pillar"/>
-    <child link="base_link"/>
-  </joint>
-  <!--joint name="pillar_to_rear_pillars" type="fixed">
-    <origin xyz="0 -0.37 0.8" rpy="0 0 0"/>
-    <parent link="support_pillar"/>
-    <child link="rear_pillars"/>
-  </joint-->
+  </joint> -->
   <!-- <joint name="vention_to_base" type="fixed">
-    <origin xyz="0 0 0.85" rpy="0 0 0"/>
+    <origin xyz="0 0 0" rpy="0 0 0"/>
     <parent link="vention_assembly"/>
     <child link="base_link"/>
-  </joint> -->
+  </joint>  -->
   <joint name="ur_to_gripper" type="fixed">
     <origin xyz="0 0 0.0" rpy="0 0 0"/>
@@ -104,7 +104,28 @@
     <child link="conveyor_base"/>
   </joint-->
-  <joint name="fixed" type="fixed">
+  <!-- <joint name="fixed" type="fixed">
       <parent link="world"/>
-      <child link="base"/>
-  </joint>
+      <child link="base_link"/>
+  </joint> -->
+  <gazebo reference="support_pillar">
+      <selfCollide>true</selfCollide>
+  </gazebo>
+  <gazebo reference="rear_pillars">
+    <selfCollide>true</selfCollide>
+  </gazebo>
+  <!-- <gazebo reference="vention_assembly">
+      <selfCollide>true</selfCollide>
+  </gazebo> -->
+  <gazebo reference="quick_change_robot_side">
+      <selfCollide>true</selfCollide>
+  </gazebo>
+  <disable_collisions link1="base_link" link2="support_pillar" reason="Adjacent" />
+  <!-- <disable_collisions link1="base_link" link2="vention_assembly" reason="Adjacent" /> -->
+  <disable_collisions link1="tool0" link2="quick_change_robot_side" reason="Adjacent" />
+  <gazebo>
+      <plugin name="ros_control" filename="libgazebo_ros_control.so">
+        <!--robotNamespace>/</robotNamespace-->
+        <!--robotSimType>gazebo_ros_control/DefaultRobotHWSim</robotSimType-->
+      </plugin>
+    </gazebo>
 </robot>
