Commit message: Gazebo and collision objects ready

File: urdf/onion_bin.urdf.xacro (robot description, xacro)
@@ -7,5 +7,5 @@
  <link name="world"/>
  <joint name="world_bin_joint" type="fixed" >
-        <origin xyz="0.1 0.6 0" rpy="0.0 0.0 0.0"/>
+        <origin xyz="0.6 -0.1 0" rpy="0.0 0.0 0.0"/>
         <parent link="world" />
         <child link="onion_bin"/>

File: urdf/ur3e_combined_gazebo.urdf.xacro (robot description, xacro)
@@ -16,5 +16,5 @@
         <origin xyz="0 0 0" rpy="0 0 0"/>
         <geometry>
-          <box size="0.15 0.15 1.2"/>
+          <box size="0.8 0.5 0.7"/>
         </geometry>
         <material name="4,4,4"/>
@@ -23,5 +23,5 @@
         <origin xyz="0 0 0" rpy="0 0 0"/>
         <geometry>
-          <box size="0.15 0.15 1.2"/>
+          <box size="0.8 0.5 0.7"/>
         </geometry>
       </collision>
@@ -36,5 +36,5 @@
         <origin xyz="0 0 0" rpy="0 0 0"/>
         <geometry>
-          <box size="0.8 0.05 1.55"/>
+          <box size="0.8 0.05 1"/>
         </geometry>
         <material name="4,4,4"/>
@@ -43,5 +43,5 @@
         <origin xyz="0 0 0" rpy="0 0 0"/>
         <geometry>
-          <box size="0.8 0.05 1.55"/>
+          <box size="0.8 0.05 1"/>
         </geometry>
       </collision>
@@ -69,15 +69,15 @@
   <!-- fix the ur robot in place -->
   <joint name="world_to_pillar" type="fixed">
-    <origin xyz="0 0 0.6" rpy="0 0 0"/>
+    <origin xyz="0 -0.15 0.35" rpy="0 0 0"/>
     <parent link="world"/>
     <child link="support_pillar"/>
   </joint>
   <joint name="pillar_to_base" type="fixed">
-  <origin xyz="0 0 0.6" rpy="0 0 0"/>
+  <origin xyz="0 0.15 0.35" rpy="0 0 0"/>
   <parent link="support_pillar"/>
   <child link="base_link"/>
   </joint>
   <joint name="pillar_to_rear_pillars" type="fixed">
-  <origin xyz="0 -0.37 0.8" rpy="0 0 0"/>
+  <origin xyz="0 -0.25 0.7" rpy="0 0 0"/>
   <parent link="support_pillar"/>
   <child link="rear_pillars"/>
