Commit message: Working on getting the demo at VOVRC working

File: urdf/ur3e_combined_collision.urdf.xacro (robot description, xacro)
@@ -82,5 +82,5 @@
   </joint-->
   <joint name="pillar_to_base" type="fixed">
-    <origin xyz="0 0 0.4" rpy="0 0 0"/>
+    <origin xyz="0 0 0.836" rpy="0 0 0"/>
     <parent link="support_pillar"/>
     <child link="base_link"/>

Commit message: Initial changes to model the VOVRC conveyor

File: urdf/ur3e_combined_collision.urdf.xacro (robot description, xacro)
@@ -20,5 +20,5 @@
         <origin xyz="0 0 0" rpy="0 0 0"/>
         <geometry>
-          <box size="0.8 0.8 0.8"/>
+          <box size="0.2 0.2 0.8"/>
         </geometry>
       </visual>
@@ -26,5 +26,5 @@
         <origin xyz="0 0 0" rpy="0 0 0"/>
         <geometry>
-          <box size="0.8 0.8 0.55"/>
+          <box size="0.2 0.2 0.55"/>
         </geometry>
       </collision>
