Commit message: All latest changes

File: onrobot_sg/models/onrobot_sg_b/sg_b.urdf (robot description, URDF)
Before this commit: robot sg-b, 2 links, 1 joints
Links:
- link quick_change_robot_side: geometry collision cylinder length=0.015 radius=0.045; visual mesh filename=package://ur3e_irl_project/onrobot_sg/models/common/Quick_C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 scale=1 1 1

File: urdf/conveyor.urdf.xacro (robot description, xacro)
@@ -1,7 +1,7 @@
 <?xml version="1.0"?>
 <robot name="conveyor_table" xmlns:xacro="http://www.ros.org/wiki/xacro">
-<!-- Author: Prasanth Suresh (ps32611@uga.edu); Description: Conveyor table to be used by ur3e -->
-<!-- Do not edit/replicate without permission -->
-<!--
+  <!-- Author: Prasanth Suresh (ps32611@uga.edu); Description: Conveyor table to be used by ur3e -->
+  <!-- Do not edit/replicate without permission -->
+  <!--
 Belt Width:15.7inch ;
 Belt Thickness:0.07inch ;
@@ -9,787 +9,784 @@
 Conveyor High:29.5inch
 -->
-  <xacro:arg name="gazebo" default="false"/>
-  <xacro:arg name="load_rollers" default="false"/>
-  <xacro:arg name="load_motors" default="false"/>
-  <xacro:arg name="load_railings" default="false"/>
+  <xacro:arg name="gazebo" default="false" />
+  <xacro:arg name="load_rollers" default="false" />
+  <xacro:arg name="load_motors" default="false" />
+  <xacro:arg name="load_railings" default="false" />
   <material name="white">
-    <color rgba="1 1 1 1"/>
+    <color rgba="1 1 1 1" />
   </material>
   <material name="black">
-    <color rgba="0 0 0 1"/>
+    <color rgba="0 0 0 1" />
   </material>
   <material name="darkgray">
-    <color rgba=".2 .2 .2 1"/>
+    <color rgba=".2 .2 .2 1" />
   </material>
   <material name="darkred">
-    <color rgba=".5 .1 .1 1"/>
+    <color rgba=".5 .1 .1 1" />
   </material>
   <material name="ur3e_red">
-    <color rgba=".5 .1 .1 1"/>
+    <color rgba=".5 .1 .1 1" />
   </material>
   <material name="ur3e_gray">
-    <color rgba="0.75294 0.75294 0.75294 1"/>
+    <color rgba="0.75294 0.75294 0.75294 1" />
   </material>
-  <link name="world"/>
+  <link name="world" />
   <joint name="world_to_frame" type="fixed">
-    <parent link="world"/>
-    <child link="frame"/>
-   <xacro:if value="$(arg gazebo)">
-    <dynamics damping="10.0" friction="5.0"/>
-   </xacro:if>
+    <parent link="world" />
+    <child link="frame" />
+    <xacro:if value="$(arg gazebo)">
+      <dynamics damping="10.0" friction="5.0" />
+    </xacro:if>
   </joint>
-    <link name="frame" type="fixed" >
-       <visual>
-	<origin rpy="0 0 0" xyz="0.5 -0.75 0" />
-  	  <geometry>
-		<mesh filename="package://ur3e_irl_project/meshes/lab_conveyor/frame.stl"/>
-	  </geometry>
-       </visual>
-	<collision>
-          <origin rpy="0 0 0" xyz="0.5 -0.75 0" />
-  	  <geometry>
-		<mesh filename="package://ur3e_irl_project/meshes/lab_conveyor/conveyor_box.stl"/>
-	  </geometry>
-	</collision>
+  <link name="frame" type="fixed">
+    <visual>
+      <origin rpy="0 0 0" xyz="0.5 -0.75 0" />
+      <geometry>
+        <mesh filename="package://ur3e_irl_project/meshes/lab_conveyor/frame.stl" />
+      </geometry>
+    </visual>
+    <collision>
+      <origin rpy="0 0 0" xyz="0.5 -0.75 0" />
+      <geometry>
+        <mesh filename="package://ur3e_irl_project/meshes/lab_conveyor/conveyor_box.stl" />
+      </geometry>
+    </collision>
     <inertial>
-       <origin rpy="0 0 0" xyz="0.01 0.75 0.46"/>
-       <mass value="29.18"/>
-      <inertia ixx="30.49" ixy="0.13" ixz="0.10" iyy="9.39" iyz="10.09" izz="22.63"/>
-      </inertial>
-    </link>
+      <origin rpy="0 0 0" xyz="0.01 0.75 0.46" />
+      <mass value="29.18" />
+      <inertia ixx="30.49" ixy="0.13" ixz="0.10" iyy="9.39" iyz="10.09" izz="22.63" />
+    </inertial>
+  </link>
   <joint name="frame_to_belt" type="fixed">
     <origin rpy="0 0 0" xyz="0.5 0 0.73" />
-    <parent link="frame"/>
-    <child link="belt"/>
-   <xacro:if value="$(arg gazebo)">
-    <dynamics damping="10.0" friction="5.0"/>
-   </xacro:if>
-   </joint>
-   <link name="belt" type="fixed" >
-       <visual>
-	<origin rpy="0 0 0" xyz="0 0 0" />
-  	  <geometry>
-		<mesh filename="package://ur3e_irl_project/meshes/lab_conveyor/belt.stl"/>
-	  </geometry>
-       </visual>
-	<collision>
-          <origin rpy="0 0 0" xyz="0 0 0" />
-  	  <geometry>
-		<mesh filename="package://ur3e_irl_project/meshes/lab_conveyor/belt.stl"/>
-	  </geometry>
-	</collision>
-    <inertial>
-       <origin rpy="0 0 0" xyz="0 0.7 0"/>
-       <mass value="1.75"/>
-      <inertia ixx="1.21" ixy="0" ixz="0" iyy="0.01" iyz="0" izz="1.2"/>
-    </inertial>
-    </link>
-<xacro:if value="$(arg load_railings)">
-<!-- The reason why these are initialized w.r.t the world frame is because
-we want floating joints above the conveyor and w.r.t the frame will not do that -->
-  <joint name="frame_railing1_joint" type="fixed" >
-        <origin xyz="0.6 0.0 0.82" rpy="0.0 0.0 0.0"/>
-        <parent link="world" />
-        <child link="railing1"/>
+    <parent link="frame" />
+    <child link="belt" />
+    <xacro:if value="$(arg gazebo)">
+      <dynamics damping="10.0" friction="5.0" />
+    </xacro:if>
   </joint>
-  <joint name="frame_railing2_joint" type="fixed" >
-        <origin xyz="0.9 0.0 0.82" rpy="0.0 0.0 0.0"/>
-        <parent link="world" />
-        <child link="railing2"/>
-  </joint>
-<link name="railing1">
+  <link name="belt" type="fixed">
+    <visual>
+      <origin rpy="0 0 0" xyz="0 0 0" />
+      <geometry>
+        <mesh filename="package://ur3e_irl_project/meshes/lab_conveyor/belt.stl" />
+      </geometry>
+    </visual>
     <collision>
-      <origin xyz="0 0 0.0" rpy="0 0 0"/>
+      <origin rpy="0 0 0" xyz="0 0 0" />
       <geometry>
-        <box size="0.01 1.5 0.01"/>-
+        <mesh filename="package://ur3e_irl_project/meshes/lab_conveyor/belt.stl" />
       </geometry>
     </collision>
-    <visual>
-      <origin xyz="0 0 0.0" rpy="0 0 0"/>
-      <geometry>
-        <box size="0.01 1.5 0.01"/>-
-      </geometry>
-    </visual>
     <inertial>
-      <origin xyz="0 0 0.0" rpy="0 0 0"/>
-      <mass value="1"/>
-      <inertia
-        ixx="1" ixy="0.0" ixz="0.0"
-        iyy="1" iyz="0.0"
-        izz="1"/>
+      <origin rpy="0 0 0" xyz="0 0.7 0" />
+      <mass value="1.75" />
+      <inertia ixx="1.21" ixy="0" ixz="0" iyy="0.01" iyz="0" izz="1.2" />
     </inertial>
   </link>
-  <gazebo reference="railing1">
+  <xacro:if value="$(arg load_railings)">
+    <!-- The reason why these are initialized w.r.t the world frame is because
+we want floating joints above the conveyor and w.r.t the frame will not do that -->
+    <joint name="frame_railing1_joint" type="fixed">
+      <origin xyz="0.6 0.0 0.82" rpy="0.0 0.0 0.0" />
+      <parent link="world" />
+      <child link="railing1" />
+    </joint>
+    <joint name="frame_railing2_joint" type="fixed">
+      <origin xyz="0.9 0.0 0.82" rpy="0.0 0.0 0.0" />
+      <parent link="world" />
+      <child link="railing2" />
+    </joint>
+    <link name="railing1">
+      <collision>
+        <origin xyz="0 0 0.0" rpy="0 0 0" />
+        <geometry>
+          <box size="0.01 1.5 0.01" />
+          -
+        </geometry>
+      </collision>
+      <visual>
+        <origin xyz="0 0 0.0" rpy="0 0 0" />
+        <geometry>
+          <box size="0.01 1.5 0.01" />
+          -
+        </geometry>
+      </visual>
+      <inertial>
+        <origin xyz="0 0 0.0" rpy="0 0 0" />
+        <mass value="1" />
+        <inertia ixx="1" ixy="0.0" ixz="0.0" iyy="1" iyz="0.0" izz="1" />
+      </inertial>
+    </link>
+    <gazebo reference="railing1">
       <mu1>0.0000001</mu1>
       <mu2>0.0000001</mu2>
-  </gazebo>
-  <link name="railing2">
-    <collision>
-      <origin xyz="0 0 0.0" rpy="0 0 0"/>
-      <geometry>
-        <box size="0.01 1.5 0.01"/>-
-      </geometry>
-    </collision>
-    <visual>
-      <origin xyz="0 0 0.0" rpy="0 0 0"/>
-      <geometry>
-        <box size="0.01 1.5 0.01"/>-
-      </geometry>
-    </visual>
-    <inertial>
-      <origin xyz="0 0 0.0" rpy="0 0 0"/>
-      <mass value="1"/>
-      <inertia
-        ixx="1" ixy="0.0" ixz="0.0"
-        iyy="1" iyz="0.0"
-        izz="1"/>
-    </inertial>
-  </link>
-  <gazebo reference="railing2">
+    </gazebo>
+    <link name="railing2">
+      <collision>
+        <origin xyz="0 0 0.0" rpy="0 0 0" />
+        <geometry>
+          <box size="0.01 1.5 0.01" />
+          -
+        </geometry>
+      </collision>
+      <visual>
+        <origin xyz="0 0 0.0" rpy="0 0 0" />
+        <geometry>
+          <box size="0.01 1.5 0.01" />
+          -
+        </geometry>
+      </visual>
+      <inertial>
+        <origin xyz="0 0 0.0" rpy="0 0 0" />
+        <mass value="1" />
+        <inertia ixx="1" ixy="0.0" ixz="0.0" iyy="1" iyz="0.0" izz="1" />
+      </inertial>
+    </link>
+    <gazebo reference="railing2">
       <mu1>0.0000001</mu1>
       <mu2>0.0000001</mu2>
+    </gazebo>
+  </xacro:if>
+  <xacro:if value="$(arg load_rollers)">
+    <joint name="frame_to_roller1" type="revolute">
+      <origin xyz="0.75 -0.7 0.73" rpy="0 0 0" />
+      <axis xyz="1 0 0" />
+      <limit lower="0.0" upper="6.28319" effort="1000.0" velocity="0.5" />
+      <parent link="frame" />
+      <child link="roller1" />
+      <xacro:if value="$(arg gazebo)">
+        <dynamics damping="10.0" friction="5.0" />
+      </xacro:if>
+    </joint>
+    <link name="roller1" type="fixed">
+      <visual>
+        <origin rpy="0 0 0" xyz="0 0 0" />
+        <geometry>
+          <mesh filename="package://ur3e_irl_project/meshes/lab_conveyor/roller.stl" />
+        </geometry>
+      </visual>
+      <collision>
+        <origin rpy="1.5708 0 0" xyz="0 0 0" />
+        <geometry>
+          <cylinder length="0.26" radius="0.04" />
+        </geometry>
+      </collision>
+      <inertial>
+        <origin rpy="0 0 0" xyz="0 0 0" />
+        <mass value="11.56" />
+        <inertia ixx="0.01" ixy="0" ixz="0" iyy="0.09" iyz="0" izz="0.09" />
+      </inertial>
+    </link>
+    <joint name="frame_to_roller2" type="revolute">
+      <origin rpy="0 0 0" xyz="0.75 -0.6 0.73" />
+      <axis xyz="1 0 0" />
+      <limit lower="0.0" upper="6.28319" effort="1000.0" velocity="0.5" />
+      <parent link="frame" />
+      <child link="roller2" />
+      <xacro:if value="$(arg gazebo)">
+        <dynamics damping="10.0" friction="5.0" />
+      </xacro:if>
+    </joint>
+    <link name="roller2" type="fixed">
+      <visual>
+        <origin rpy="0 0 0" xyz="0 0 0" />
+        <geometry>
+          <mesh filename="package://ur3e_irl_project/meshes/lab_conveyor/roller.stl" />
+        </geometry>
+      </visual>
+      <collision>
+        <origin rpy="1.5708 0 0" xyz="0 0 0" />
+        <geometry>
+          <cylinder length="0.26" radius="0.04" />
+        </geometry>
+      </collision>
+      <inertial>
+        <origin rpy="0 0 0" xyz="0 0 0" />
+        <mass value="11.56" />
+        <inertia ixx="0.01" ixy="0" ixz="0" iyy="0.09" iyz="0" izz="0.09" />
+      </inertial>
+    </link>
+    <joint name="frame_to_roller3" type="revolute">
+      <origin rpy="0 0 0" xyz="0.75 -0.5 0.73" />
+      <axis xyz="1 0 0" />
+      <limit lower="0.0" upper="6.28319" effort="1000.0" velocity="0.5" />
+      <parent link="frame" />
+      <child link="roller3" />
+      <xacro:if value="$(arg gazebo)">
+        <dynamics damping="10.0" friction="5.0" />
+      </xacro:if>
+    </joint>
+    <link name="roller3" type="fixed">
+      <visual>
+        <origin rpy="0 0 0" xyz="0 0 0" />
+        <geometry>
+          <mesh filename="package://ur3e_irl_project/meshes/lab_conveyor/roller.stl" />
+        </geometry>
+      </visual>
+      <collision>
+        <origin rpy="1.5708 0 0" xyz="0 0 0" />
+        <geometry>
+          <cylinder length="0.26" radius="0.04" />
+        </geometry>
+      </collision>
+      <inertial>
+        <origin rpy="0 0 0" xyz="0 0 0" />
+        <mass value="11.56" />
+        <inertia ixx="0.01" ixy="0" ixz="0" iyy="0.09" iyz="0" izz="0.09" />
+      </inertial>
+    </link>
+    <joint name="frame_to_roller4" type="revolute">
+      <origin rpy="0 0 0" xyz="0.75 -0.4 0.73" />
+      <axis xyz="1 0 0" />
+      <limit lower="0.0" upper="6.28319" effort="1000.0" velocity="0.5" />
+      <parent link="frame" />
+      <child link="roller4" />
+      <xacro:if value="$(arg gazebo)">
+        <dynamics damping="10.0" friction="5.0" />
+      </xacro:if>
+    </joint>
+    <link name="roller4" type="fixed">
+      <visual>
+        <origin rpy="0 0 0" xyz="0 0 0" />
+        <geometry>
+          <mesh filename="package://ur3e_irl_project/meshes/lab_conveyor/roller.stl" />
+        </geometry>
+      </visual>
+      <collision>
+        <origin rpy="1.5708 0 0" xyz="0 0 0" />
+        <geometry>
+          <cylinder length="0.26" radius="0.04" />
+        </geometry>
+      </collision>
+      <inertial>
+        <origin rpy="0 0 0" xyz="0 0 0" />
+        <mass value="11.56" />
+        <inertia ixx="0.01" ixy="0" ixz="0" iyy="0.09" iyz="0" izz="0.09" />
+      </inertial>
+    </link>
+    <joint name="frame_to_roller5" type="revolute">
+      <origin rpy="0 0 0" xyz="0.75 -0.3 0.73" />
+      <axis xyz="1 0 0" />
+      <limit lower="0.0" upper="6.28319" effort="1000.0" velocity="0.5" />
+      <parent link="frame" />
+      <child link="roller5" />
+      <xacro:if value="$(arg gazebo)">
+        <dynamics damping="10.0" friction="5.0" />
+      </xacro:if>
+    </joint>
+    <link name="roller5" type="fixed">
+      <visual>
+        <origin rpy="0 0 0" xyz="0 0 0" />
+        <geometry>
+          <mesh filename="package://ur3e_irl_project/meshes/lab_conveyor/roller.stl" />
+        </geometry>
+      </visual>
+      <collision>
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
File: urdf/ur3e_combined_collision.urdf.xacro (robot description, xacro)
@@ -6,4 +6,7 @@
   <!--xacro:include filename="$(find ur3e_irl_project)/urdf/conveyor_g_path.urdf.xacro"/-->
   <xacro:include filename="$(find ur3e_irl_project)/onrobot_sg/models/onrobot_sg_b/sg_b.urdf"/>
+  <material name="ur3e_gray">
+    <color rgba="0.75294 0.75294 0.75294 1" />
+  </material>
   <link name="world" />
   <link name="support_pillar">
@@ -14,9 +17,9 @@
       </inertial>
       <visual>
+        <material name="ur3e_gray"/>
         <origin xyz="0 0 0" rpy="0 0 0"/>
         <geometry>
           <box size="0.8 0.8 0.8"/>
         </geometry>
-        <material name="4,4,4"/>
       </visual>
       <collision>
@@ -34,9 +37,9 @@
       </inertial>
       <visual>
+        <material name="ur3e_gray"/>
         <origin xyz="0 0 0" rpy="0 0 0"/>
         <geometry>
           <box size="0.8 0.05 1.55"/>
         </geometry>
-        <material name="4,4,4"/>
       </visual>
       <collision>

File: urdf/ur3e_combined_gazebo.urdf.xacro (robot description, xacro)
@@ -47,4 +47,8 @@
       </collision>
   </link>
+  <xacro:include filename="$(find realsense2_description)/urdf/_d435.urdf.xacro" />
+  <xacro:sensor_d435 name="camera" topics_ns="camera" parent="world" publish_pointcloud="true">
+    <origin xyz="-0.25 -0.36 1.25" rpy="0 0.7 1.5" />
+  </xacro:sensor_d435>
    <!-- <link name="vention_assembly">
       <inertial>

Commit message: Minor corrections in collisions

File: onrobot_sg/models/onrobot_sg_b/sg_b.urdf (robot description, URDF)
Before this commit: robot sg-b, 2 links, 1 joints
Links:
- link gripper: geometry collision cylinder length=0.15 radius=0.049; visual mesh filename=package://ur3e_irl_project/onrobot_sg/models/onrobot_sg_b/m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 scale=1 1 1

File: urdf/ur3e_combined_collision.urdf.xacro (robot description, xacro)
@@ -97,5 +97,5 @@
   </joint-->
   <joint name="ur_to_gripper" type="fixed">
-    <origin xyz="0 0 0.0" rpy="0 0 0"/>
+    <origin xyz="0 0.0 0.0" rpy="0 0 0"/>
     <parent link="tool0"/>
     <child link="quick_change_robot_side"/>

Commit message: All changes

File: onrobot_sg/models/onrobot_sg_b/sg_b.urdf (robot description, URDF)
Before this commit: robot sg-b, 2 links, 1 joints
Links:
- link gripper: geometry collision cylinder length=0.10 radius=0.049; visual mesh filename=package://ur3e_irl_project/onrobot_sg/models/onrobot_sg_b/m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 scale=1 1 1

File: urdf/ur3e_combined_collision.urdf.xacro (robot description, xacro)
@@ -26,5 +26,5 @@
         <origin xyz="0 0 0" rpy="0 0 0"/>
         <geometry>
-          <box size="0.8 0.8 0.8"/>
+          <box size="0.8 0.8 0.55"/>
         </geometry>
       </collision>
